File: Vibration_Board/Vibration_Board.kicad_sch (KiCad schematic)
At the start: 0 parts

Commit message: everything added
Other:
- sheet Connectors ports: added ACCELER_CS5, ACCELER_CS6, ACCELER_CS7, ACCELER_CS8, MISO_2, MOSI_2, SCK_2; removed none
- sheet MCU ports: added ACCELERMETER_CS5, ACCELERMETER_CS6, ACCELERMETER_CS7, ACCELERMETER_CS8, CUR_SEN, MISO_2, MOSI_2, SCK_2, TEMP_RESET; removed none
