File: Vibration_Board/Vibration_Board.kicad_pcb (KiCad board)
At the start: 4 copper layers, 100 x 60 mm, 47 parts, among them J1 Debugging Connector, J10 Conn_01x06_Pin, J11 Conn_01x06_Pin, J2 Micro_SD_Card, J3 Conn_01x06_Pin, J4 Conn_01x06_Pin, J5 G125-MH104M4-04AD000P, J6 Conn_01x06_Pin, J7 Conn_01x06_Pin, J8 Conn_01x06_Pin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

Commit message: build files,bom and jlc bom
Parts:
- added G***: LOGO, LOGO, B.Cu at (26.2, 43.8)
Other:
- board text added: "Vibration Board V1 Rajeev Persaud June 24th 2026 My head hurts very badly"

Commit message: fixes from review
Parts:
- added 3V3D1: 4952, 1726750413:KEYSTONE_4952, F.Cu at (83.5, 42.5)
- added 5V1: 4952, 1726750413:KEYSTONE_4952, F.Cu at (96.2, 34.2)
- added MISO1: 4952, 1726750413:KEYSTONE_4952, F.Cu at (62.2, 60.0)
- added MISO2: 4952, 1726750413:KEYSTONE_4952, F.Cu at (37.8, 30.2)
- added MOSI1: 4952, 1726750413:KEYSTONE_4952, F.Cu at (41.2, 61.0)
- added MOSI2: 4952, 1726750413:KEYSTONE_4952, F.Cu at (41.8, 26.2)
- added R10: 220R, Resistor_SMD:R_0805_2012Metric_Pad1.20x1.40mm_HandSolder, F.Cu at (61.5, 20.0)
- added R11: 220R, Resistor_SMD:R_0805_2012Metric_Pad1.20x1.40mm_HandSolder, F.Cu at (61.8, 24.2)
- added R12: 220R, Resistor_SMD:R_0805_2012Metric_Pad1.20x1.40mm_HandSolder, F.Cu at (62.8, 26.5)
- added R13: 220R, Resistor_SMD:R_0805_2012Metric_Pad1.20x1.40mm_HandSolder, F.Cu at (66.5, 25.2)
- added R2: 4.7KR, Resistor_SMD:R_0805_2012Metric_Pad1.20x1.40mm_HandSolder, B.Cu at (51.2, 31.0)
- added R8: 4.7KR, Resistor_SMD:R_0805_2012Metric_Pad1.20x1.40mm_HandSolder, B.Cu at (51.2, 33.2)
- added R9: 220R, Resistor_SMD:R_0805_2012Metric_Pad1.20x1.40mm_HandSolder, F.Cu at (62.0, 17.2)
- added RX1: 4952, 1726750413:KEYSTONE_4952, F.Cu at (83.0, 51.8)
- added SCK1: 4952, 1726750413:KEYSTONE_4952, F.Cu at (75.0, 56.0)
- added SCK2: 4952, 1726750413:KEYSTONE_4952, F.Cu at (84.8, 31.0)
- added TX1: 4952, 1726750413:KEYSTONE_4952, F.Cu at (86.5, 47.2)
- R3, R4, R5, R6, R7: value R_US -> 220R
Connections:
- J4 pad 2: /Connectors/MOSI_2 -> +3.3VD
- J4 pad 3: /Connectors/MISO_2 -> /Connectors/MOSI_2
- J4 pad 4: /Connectors/SCK_2 -> /Connectors/MISO_2
- J4 pad 5: +3.3VD -> /Connectors/SCK_2
- J6 pad 2: /MOSI -> +3.3VD
- J6 pad 3: /MISO -> /MOSI
- J6 pad 4: /SCK -> /MISO
- J6 pad 5: +3.3VD -> /SCK
- J7 pad 2: /MOSI -> +3.3VD
- J7 pad 3: /MISO -> /MOSI
- J7 pad 4: /SCK -> /MISO
- J7 pad 5: +3.3VD -> /SCK
Routing:
- net +3.3VD: track 50.1 -> 59.7 mm, vias 37 -> 44
- net /Connectors/MISO_2: track 92.6 -> 99.4 mm
- net /Connectors/MOSI_2: track 90.4 -> 96.7 mm
- net /TX: track 37.6 -> 43.6 mm
- net /RX: track 38.2 -> 44.0 mm
- net /Connectors/SCK_2: track 96.3 -> 101.4 mm
- net GND: track 17.8 -> 22.5 mm, vias 42 -> 48
- net /MISO: track 97.6 -> 101.7 mm
- net /Connectors/DATA1: track 25.1 -> 28.6 mm, vias 1 -> 2
- net +5V: track 39.3 -> 42.6 mm
- net /Connectors/SD_CS: track 18.9 -> 21.9 mm, vias 1 -> 2
- net /MOSI: track 90.2 -> 93.1 mm
- net /Connectors/DATA4: track 18.4 -> 21.2 mm, vias 1 -> 2
- net /SCK: track 106.1 -> 108.5 mm
- net /Connectors/DATA2: track 25.5 -> 27.6 mm, vias 1 -> 2
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
Commit message: layer problem for exporting
Routing:
- added copper zone on In2.Cu, net GND
Changed lines of the file:
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@@
 		(tags "capacitor handsolder")
 		(property "Reference" "C31"
-			(at 2.725 -0.05 180)
+			(at 0.775 1.8 270)
 			(layer "F.SilkS")
 			(effects
@@
 		(at 83.5 42.5)
 		(property "Reference" "3V3D1"
-			(at 0.127 -2.3114 0)
+			(at -3.5 -0.75 0)
 			(layer "F.SilkS")
 			(effects
@@
 			)
 		)
+	)
+	(zone
+		(net 1)
+		(net_name "GND")
+		(layer "In2.Cu")
+		(hatch edge 0.5)
+		(priority 4)
+		(connect_pads
+			(clearance 0.5)
+		)
+		(min_thickness 0.25)
+		(filled_areas_thickness no)
+		(fill yes
+			(thermal_gap 0.5)
+			(thermal_bridge_width 0.5)
+		)
+		(polygon
+			(pts
+				(xy 113.25 13.25) (xy 113.5 13.5) (xy 113.5 73.75) (xy 12.5 73.75) (xy 12.5 13.25)
+			)
+		)
