File: Vibration_Board/Connectors.kicad_sch (KiCad schematic)
At the start: 10 parts, among them J1 Debugging Connector, J2 Micro_SD_Card, J3 Gecko Connector, J4 Gecko Connector, J5 G125-MH104M4-04AD000P, J6 Gecko Connector, J7 Gecko Connector, U10 MCP2562

Commit message: everything added
Parts:
- added J10, J11, J8, J9: Conn_01x06_Pin, jst:CONN6_S6B-PH_JST, symbol Connector:Conn_01x06_Pin
- C3, C4: footprint Capacitor_SMD:C_0603_1608Metric_Pad1.08x0.95mm_HandSolder -> Capacitor_SMD:C_0805_2012Metric_Pad1.18x1.45mm_HandSolder
- J3, J4, J6, J7: value Gecko Connector -> Conn_01x06_Pin; footprint G125-MH104M4-04AD000P:connector_Harwin_M80-5000642 -> jst:CONN6_S6B-PH_JST
Connections:
- net +3.3VD: now also J10.2 (Pin_2), J11.2 (Pin_2), J8.2 (Pin_2), J9.2 (Pin_2)
- net GND: now also J10.1 (Pin_1), J11.1 (Pin_1), J8.1 (Pin_1), J9.1 (Pin_1)
- net MISO: now also J11.4 (Pin_4), J8.4 (Pin_4); no longer J3.4 (Pin_4), J4.3 (Pin_3)
- net MOSI: now also J11.3 (Pin_3), J8.3 (Pin_3); no longer J3.3 (Pin_3), J4.2 (Pin_2)
- net SCK: now also J11.5 (Pin_5), J8.5 (Pin_5); no longer J3.5 (Pin_5), J4.4 (Pin_4)
- new net ACCELER_CS5: J8.6 (Pin_6)
- new net ACCELER_CS6: J9.6 (Pin_6)
- new net ACCELER_CS7: J10.6 (Pin_6)
- new net ACCELER_CS8: J11.6 (Pin_6)
- new net MISO_2: J10.4 (Pin_4), J3.4 (Pin_4), J4.3 (Pin_3), J9.4 (Pin_4)
- new net MOSI_2: J10.3 (Pin_3), J3.3 (Pin_3), J4.2 (Pin_2), J9.3 (Pin_3)
- new net SCK_2: J10.5 (Pin_5), J3.5 (Pin_5), J4.4 (Pin_4), J9.5 (Pin_5)
Other:
- moved on the sheet: J2

Commit message: fixes from review
Parts:
- added R10, R11, R12, R13, R9: 220R, Resistor_SMD:R_0805_2012Metric_Pad1.20x1.40mm_HandSolder, symbol Device:R_US
Connections:
- net +3.3VD: now also J4.2 (Pin_2), J6.2 (Pin_2), J7.2 (Pin_2), R10.1, R11.1, R12.1, R13.1, R9.1; no longer J4.5 (Pin_5), J6.5 (Pin_5), J7.5 (Pin_5)
- net DATA1: now also R9.2
- net DATA2: now also R10.2
- net DATA3: now also R13.2
- net DATA4: now also R12.2
- net MISO: now also J6.4 (Pin_4), J7.4 (Pin_4); no longer J6.3 (Pin_3), J7.3 (Pin_3)
- net MISO_2: now also J4.4 (Pin_4); no longer J4.3 (Pin_3)
- net MOSI: now also J6.3 (Pin_3), J7.3 (Pin_3); no longer J6.2 (Pin_2), J7.2 (Pin_2)
- net MOSI_2: now also J4.3 (Pin_3); no longer J4.2 (Pin_2)
- net SCK: now also J6.5 (Pin_5), J7.5 (Pin_5); no longer J6.4 (Pin_4), J7.4 (Pin_4)
- net SCK_2: now also J4.5 (Pin_5); no longer J4.4 (Pin_4)
- net SD_CS: now also R11.2
