File: Vibration_Board/MCU.kicad_sch (KiCad schematic)
At the start: 25 parts, among them U4 STM32H745ZIT6

Commit message: everything added
Parts:
- removed C11, C12, C13, C14, C15, C16, C17, C18: 1uF, Capacitor_SMD:C_0805_2012Metric_Pad1.18x1.45mm_HandSolder, symbol Device:C
- removed U4: STM32H745ZIT6, STM32H745ZIT6:LQFP144, symbol STM32H745ZIT6:STM32H745ZIT6
- added U4: STM32H750VBT6TR, STM32H745ZIT6:QFP50P1600X1600X160-100N, symbol STM32H750VBT6TR:STM32H750VBT6TR
- R3, R4, R5, R6, R7: value R_US -> 220R
Connections:
- net +3.3VD: now also U4.100 (VDD), U4.11 (VDD), U4.20 (VREF+), U4.21 (VDDA), U4.27 (VDD), U4.50 (VDD), U4.75 (VDD); no longer C10.1
- net ACCEROMETER_CS1: now also U4.32 (PC4/DFSDM_CKIN2/I2S1_MCK/SPDIFRX_IN2/ETH_MII_RXD0/ETH_RMII_RXD0/FMC_SDNE0/EVENTOUT/ADC12_INP4/OPAMP1_VOUT/COMP_1_INM)
- net ACCEROMETER_CS2: now also U4.33 (PC5/SAI1_D3/DFSDM_DATIN2/SPDIFRX_IN3/SAI4_D3/ETH_MII_RXD1/ETH_RMII_RXD1/FMC_SDCKE0/COMP_1_OUT/EVENTOUT/ADC12_INN4/ADC12_INP8/OPAMP1_VINM)
- net ACCEROMETER_CS3: now also U4.34 (PB0/TIM1_CH2N/TIM3_CH3/TIM8_CH2N/DFSDM_CKOUT/UART4_CTS/LCD_R3/OTG_HS_ULPI_D1/ETH_MII_RXD2/LCD_G1/EVENTOUT/ADC12_INN5/ADC12_INP9/OPAMP1_VINP/COMP_1_INP)
- net ACCEROMETER_CS4: now also U4.85 (PD4/HRTIM_FLT3/SAI3_FS_A/USART2_RTS/FDCAN1_RXFD_MODE/FMC_NOE/EVENTOUT)
- net GND: now also U4.10 (VSS), U4.19 (VSSA), U4.26 (VSS), U4.49 (VSS), U4.74 (VSS), U4.99 (VSS)
- net I2C_ALERT: now also U4.91 (PB5/TIM17_BKIN/TIM3_CH2/HRTIM_EEV7/I2C1_SMBA/SPI1_MOSI/I2S1_SDO/I2C4_SMBA/SPI3_MOSI/I2S3_SDO/SPI6_MOSI/FDCAN2_RX/OTG_HS_ULPI_D7/ETH_PPS_OUT/FMC_SDCKE1/DCMI_D10/UART5_RX/EVENTOUT)
- net I2C_DATA: now also U4.93 (PB7/TIM17_CH1N/TIM4_CH2/HRTIM_EEV9/I2C1_SDA/I2C4_SDA/USART1_RX/LPUART1_RX/FDCAN2_TXFD_MODE/DFSDM_CKIN5/FMC_NL/DCMI_VSYNC/EVENTOUT)
- net I2C_SCK: now also U4.92 (PB6/TIM16_CH1N/TIM4_CH1/HRTIM_EEV8/I2C1_SCL/HDMI_CEC/I2C4_SCL/USART1_TX/LPUART1_TX/FDCAN2_TX/QUADSPI_BK1_NCS/DFSDM_DATIN5/FMC_SDNE1/DCMI_D5/UART5_TX/EVENTOUT)
- net MCLK_IN: now also U4.12 (PH0-OSC_IN/EVENTOUT/OSC_IN)
- net MCLK_OUT: now also U4.13 (PH1-OSC_OUT/EVENTOUT/OSC_OUT)
- net MCLR: now also U4.94 (BOOT0)
- net MISO: now also U4.30 (PA6/TIM1_BKIN/TIM3_CH1/TIM8_BKIN/SPI1_MISO/I2S1_SDI/SPI6_MISO/TIM13_CH1/TIM8_BKIN_COMP12/MDIOS_MDC/TIM1_BKIN_COMP12/DCMI_PIXCLK/LCD_G2/EVENTOUT/ADC12_INP3)
- net MOSI: now also U4.31 (PA7/TIM1_CH1N/TIM3_CH2/TIM8_CH1N/SPI1_MOSI/I2S1_SDO/SPI6_MOSI/TIM14_CH1/ETH_MII_RX_DV/ETH_RMII_CRS_DV/FMC_SDNWE/EVENTOUT/ADC12_INN3/ADC12_INP7/OPAMP1_VINM)
- net PGC: now also U4.76 (PA14/JTCK-SWCLK/EVENTOUT)
- net PGD: now also U4.72 (PA13/JTMS-SWDIO/EVENTOUT)
- net RX: now also U4.70 (PA11/TIM1_CH4/HRTIM_CHD1/LPUART1_CTS/SPI2_NSS/I2S2_WS/UART4_RX/USART1_CTS_NSS/FDCAN1_RX/OTG_FS_DM/LCD_R4/EVENTOUT)
- net SCK: now also U4.29 (PA5/TIM2_CH1/TIM2_ETR/TIM8_CH1N/SPI1_SCK/I2S1_CK/SPI6_SCK/OTG_HS_ULPI_CK/LCD_R4/EVENTOUT/ADC12_INN18/ADC12_INP19/DAC1_OUT2)
- net SD_CK: now also U4.80 (PC12/TRACED3/HRTIM_EEV2/SPI3_MOSI/I2S3_SDO/USART3_CK/UART5_TX/SDMMC1_CK/DCMI_D9/EVENTOUT)
- net SD_CS: now also U4.83 (PD2/TRACED2/TIM3_ETR/UART5_RX/SDMMC1_CMD/DCMI_D11/EVENTOUT)
- net SD_DATA0: now also U4.65 (PC8/TRACED1/HRTIM_CHB1/TIM3_CH3/TIM8_CH3/USART6_CK/UART5_RTS/FMC_NE2/FMC_NCE/SWPMI_RX/SDMMC1_D0/DCMI_D2/EVENTOUT)
- net SD_DATA1: now also U4.66 (PC9/MCO2/TIM3_CH4/TIM8_CH4/I2C3_SDA/I2S_CKIN/UART5_CTS/QUADSPI_BK1_IO0/LCD_G3/SWPMI_SUSPEND/SDMMC1_D1/DCMI_D3/LCD_B2/EVENTOUT)
- net SD_DATA2: now also U4.78 (PC10/HRTIM_EEV1/DFSDM_CKIN5/SPI3_SCK/I2S3_CK/USART3_TX/UART4_TX/QUADSPI_BK1_IO1/SDMMC1_D2/DCMI_D8/LCD_R2/EVENTOUT)
- net SD_DATA3: now also U4.79 (PC11/HRTIM_FLT2/DFSDM_DATIN5/SPI3_MISO/I2S3_SDI/USART3_RX/UART4_RX/QUADSPI_BK2_NCS/SDMMC1_D3/DCMI_D4/EVENTOUT)
- net TX: now also U4.71 (PA12/TIM1_ETR/HRTIM_CHD2/LPUART1_RTS/SPI2_SCK/I2S2_CK/UART4_TX/USART1_RTS/SAI2_FS_B/FDCAN1_TX/OTG_FS_DP/LCD_R5/EVENTOUT)
- net at R7.2: now also U4.1 (PE2/TRACECLK/SAI1_CK1/SPI4_SCK/SAI1_MCLK_A/SAI4_MCLK_A/QUADSPI_BK1_IO2/SAI4_CK1/ETH_MII_TXD3/FMC_A23/EVENTOUT)
- net at R6.2: now also U4.2 (PE3/TRACED0/TIM15_BKIN/SAI1_SD_B/SAI4_SD_B/FMC_A19/EVENTOUT)
- net at R5.2: now also U4.3 (PE4/TRACED1/SAI1_D2/DFSDM_DATIN3/TIM15_CH1N/SPI4_NSS/SAI1_FS_A/SAI4_FS_A/SAI4_D2/FMC_A20/DCMI_D4/LCD_B0/EVENTOUT)
- net at R4.2: now also U4.4 (PE5/TRACED2/SAI1_CK2/DFSDM_CKIN3/TIM15_CH1/SPI4_MISO/SAI1_SCK_A/SAI4_SCK_A/SAI4_CK2/FMC_A21/DCMI_D6/LCD_G0/EVENTOUT)
- net at R3.2: now also U4.5 (PE6/TRACED3/TIM1_BKIN2/SAI1_D1/TIM15_CH2/SPI4_MOSI/SAI1_SD_A/SAI4_SD_A/SAI4_D1/SAI2_MCK_B/TIM1_BKIN2_COMP12/FMC_A22/DCMI_D7/LCD_G1/EVENTOUT)
- new net: C10.1, U4.14 (~{RST})
- new net ACCELERMETER_CS5: U4.36 (PB2/SAI1_D1/DFSDM_CKIN1/SAI1_SD_A/SPI3_MOSI/I2S3_SDO/SAI4_SD_A/QUADSPI_CLK/SAI4_D1/ETH_TX_ER/EVENTOUT/COMP_1_INP/RTC_OUT)
- new net ACCELERMETER_CS6: U4.77 (PA15/JTDI/TIM2_CH1/TIM2_ETR/HRTIM_FLT1/HDMI_CEC/SPI1_NSS/I2S1_WS/SPI3_NSS/I2S3_WS/SPI6_NSS/UART4_RTS/UART7_TX/EVENTOUT)
- new net ACCELERMETER_CS7: U4.38 (PE8/TIM1_CH1N/DFSDM_CKIN2/UART7_TX/QUADSPI_BK2_IO1/FMC_D5/FMC_DA5/COMP_2_OUT/EVENTOUT/OPAMP2_VINM)
- new net ACCELERMETER_CS8: U4.39 (PE9/TIM1_CH1/DFSDM_CKOUT/UART7_RTS/QUADSPI_BK2_IO2/FMC_D6/FMC_DA6/EVENTOUT/OPAMP2_VINP/COMP_2_INP)
- new net CUR_SEN: U4.28 (PA4/TIM5_ETR/SPI1_NSS/I2S1_WS/SPI3_NSS/I2S3_WS/USART2_CK/SPI6_NSS/OTG_HS_SOF/DCMI_HSYNC/LCD_VSYNC/EVENTOUT/ADC12_INP18/DAC1_OUT1)
- new net MISO_2: U4.90 (PB4/NJTRST/TIM16_BKIN/TIM3_CH1/HRTIM_EEV6/SPI1_MISO/I2S1_SDI/SPI3_MISO/I2S3_SDI/SPI2_NSS/I2S2_WS/SPI6_MISO/SDMMC2_D3/UART7_TX/EVENTOUT)
- new net MOSI_2: U4.87 (PD6/SAI1_D1/DFSDM_CKIN4/DFSDM_DATIN1/SPI3_MOSI/I2S3_SDO/SAI1_SD_A/USART2_RX/SAI4_SD_A/FDCAN2_RXFD_MODE/SAI4_D1/SDMMC2_CK/FMC_NWAIT/DCMI_D10/LCD_B2/EVENTOUT)
- new net SCK_2: U4.89 (PB3/JTDO/TRACESWO/TIM2_CH2/HRTIM_FLT4/SPI1_SCK/I2S1_CK/SPI3_SCK/I2S3_CK/SPI6_SCK/SDMMC2_D2/UART7_RX/EVENTOUT)
- new net TEMP_RESET: U4.98 (PE1/LPTIM1_IN2/HRTIM_SCOUT/UART8_TX/FDCAN1_TXFD_MODE/FMC_NBL1/DCMI_D3/EVENTOUT)
- new net VCAP: U4.48 (VCAP), U4.73 (VCAP)
- no-connect marks 0 -> 49
Other:
- moved on the sheet: D2, D3, D4, D5, D6, R3, R4, R5, R6, R7

Commit message: fixes from review
Parts:
- added MISO1, MISO2, MOSI1, MOSI2, RX1, SCK1, SCK2, TX1: 4952, 1726750413:KEYSTONE_4952, symbol ${KIPRJMOD}:4952
Connections:
- net MISO: now also MISO1.TP
- net MISO_2: now also MISO2.TP
- net MOSI: now also MOSI1.TP
- net MOSI_2: now also MOSI2.TP
- net RX: now also RX1.TP
- net SCK: now also SCK1.TP
- net SCK_2: now also SCK2.TP
- net TX: now also TX1.TP
