File: Vibration_Board/Power.kicad_sch (KiCad schematic)
At the start: 12 parts, among them U2 INA180A1, U3 SPX3819M5-L-3-3

Commit message: everything added
Changed lines of the file:
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@@
+	)
+	(junction
+		(at 129.54 82.55)
+		(diameter 0)
+		(color 0 0 0 0)
 	)
 	(junction
@@
 	(wire
 		(pts
+			(xy 129.54 82.55) (xy 124.46 82.55)
+		)
+		(stroke
+			(width 0)
+			(type default)
+		)
+	)
+	(wire
+		(pts
 			(xy 147.32 107.95) (xy 151.13 107.95)
 		)
@@
 	(wire
 		(pts
-			(xy 124.46 82.55) (xy 170.18 82.55)
-		)
-		(stroke
-			(width 0)
-			(type default)
-		)
-	)
-	(wire
-		(pts
 			(xy 124.46 110.49) (xy 124.46 82.55)
 		)
@@
 	(wire
 		(pts
-			(xy 124.46 53.34) (xy 124.46 82.55)
+			(xy 129.54 54.61) (xy 129.54 82.55)
 		)
 		(stroke
@@
 		(pts
 			(xy 170.18 82.55) (xy 179.07 82.55)
+		)
+		(stroke
+			(width 0)
+			(type default)
+		)
+	)
+	(wire
+		(pts
+			(xy 129.54 82.55) (xy 170.18 82.55)
 		)
 		(stroke
@@
 	(symbol
 		(lib_id "power:+5V")
-		(at 124.46 53.34 0)
+		(at 129.54 54.61 0)
 		(unit 1)
 		(exclude_from_sim no)
@@
 		(fields_autoplaced yes)
 		(property "Reference" "#PWR01"
-			(at 124.46 57.15 0)
+			(at 129.54 58.42 0)
 			(effects
 				(font
@@
 		)
 		(property "Value" "+5V"
-			(at 124.46 48.26 0)
+			(at 129.54 49.53 0)
 			(effects
 				(font
@@
 		)
 		(property "Footprint" ""
-			(at 124.46 53.34 0)
+			(at 129.54 54.61 0)
 			(effects
 				(font
@@
 		)
 		(property "Datasheet" ""
-			(at 124.46 53.34 0)
+			(at 129.54 54.61 0)
 			(effects
 				(font
@@
 		)
 		(property "Description" "Power symbol creates a global label with name \"+5V\""
-			(at 124.46 53.34 0)
-			(effects
-				(font
+			(at 129.54 54.61 0)
+			(effects
+				(font

Commit message: fixes from review
Parts:
- added 3V3D1, 5V1: 4952, 1726750413:KEYSTONE_4952, symbol ${KIPRJMOD}:4952
Connections:
- net +3.3VD: now also 3V3D1.TP
- net +5V: now also 5V1.TP
