File: Vibration_Board/Sensor.kicad_sch (KiCad schematic)
At the start: 1 part, among them U1 SHT31-DIS-B2.5KS

Commit message: everything added
Changed lines of the file:
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@@
 	(paper "A4")
-	(junction
-		(at 107.95 36.83)
-		(diameter 0)
-		(color 0 0 0 0)
-	)
 	(junction
 		(at 107.95 34.29)
@@
 	(wire
 		(pts
-			(xy 88.9 36.83) (xy 107.95 36.83)
-		)
-		(stroke
-			(width 0)
-			(type default)
-		)
-	)
-	(wire
-		(pts
 			(xy 34.29 34.29) (xy 43.18 34.29)
 		)
@@
 	(wire
 		(pts
-			(xy 107.95 34.29) (xy 107.95 36.83)
+			(xy 107.95 34.29) (xy 107.95 44.45)
+		)
+		(stroke
+			(width 0)
+			(type default)
+		)
+	)
+	(wire
+		(pts
+			(xy 107.95 31.75) (xy 107.95 34.29)
+		)
+		(stroke
+			(width 0)
+			(type default)
+		)
+	)
+	(wire
+		(pts
+			(xy 116.84 36.83) (xy 88.9 36.83)
 		)
 		(stroke
@@
 	(wire
 		(pts
+			(xy 116.84 45.72) (xy 116.84 36.83)
+		)
+		(stroke
+			(width 0)
+			(type default)
+		)
+	)
+	(wire
+		(pts
 			(xy 30.48 36.83) (xy 43.18 36.83)
 		)
@@
 	(wire
 		(pts
-			(xy 107.95 31.75) (xy 107.95 34.29)
-		)
-		(stroke
-			(width 0)
-			(type default)
-		)
-	)
-	(wire
-		(pts
 			(xy 88.9 41.91) (xy 119.38 41.91)
 		)
@@
 		(pts
 			(xy 88.9 34.29) (xy 107.95 34.29)
-		)
-		(stroke
-			(width 0)
-			(type default)
-		)
-	)
-	(wire
-		(pts
-			(xy 107.95 36.83) (xy 107.95 44.45)
 		)
 		(stroke
@@
 					(unit 1)
 				)
+			)
+		)
+	)
+	(symbol
+		(lib_id "power:GND")
+		(at 116.84 45.72 0)
+		(unit 1)
+		(exclude_from_sim no)
+		(in_bom yes)
+		(on_board yes)
+		(dnp no)
+		(fields_autoplaced yes)
+		(property "Reference" "#PWR021"
+			(at 116.84 52.07 0)
+			(effects
+				(font
+					(size 1.27 1.27)
+				)
+				(hide yes)
+			)
+		)
+		(property "Value" "GND"
+			(at 116.84 50.8 0)
+			(effects
+				(font
+					(size 1.27 1.27)
+				)
+			)
+		)
+		(property "Footprint" ""
+			(at 116.84 45.72 0)
+			(effects
+				(font
+					(size 1.27 1.27)
+				)
+				(hide yes)
+			)
+		)
+		(property "Datasheet" ""
+			(at 116.84 45.72 0)
+			(effects
+				(font
+					(size 1.27 1.27)
+				)
+				(hide yes)
+			)
+		)
+		(property "Description" "Power symbol creates a global label with name \"GND\" , ground"
+			(at 116.84 45.72 0)
+			(effects
+				(font
+					(size 1.27 1.27)
+				)
+				(hide yes)
+			)
+		)
+		(pin "1"
+		)
+		(instances
+			(project ""
+				(path "/a253d658-fd52-4305-b7af-3d5656162b72/a7cddbac-d981-4220-bd5e-99b0b94e3860"
+					(reference "#PWR021")
+					(unit 1)
+				)

Commit message: fixes from review
Parts:
- added R2, R8: 4.7KR, Resistor_SMD:R_0805_2012Metric_Pad1.20x1.40mm_HandSolder, symbol Device:R_US
Connections:
- net +3.3VD: now also R2.1, R8.1
- net I2C_CLK: now also R2.2
- net I2C_DATA: now also R8.2
